File: Watch.kicad_pcb (KiCad board)
At the start: 2 copper layers, 0 parts

Commit message: session 2
Parts:
- added BT1: Battery_Cell, Battery:BatteryHolder_Keystone_1060_1x2032, B.Cu at (177.4, 97.5)
- added C1: 1uF, Capacitor_SMD:C_0603_1608Metric, F.Cu at (172.0, 103.5)
- added C10: 10pF, Capacitor_SMD:C_0603_1608Metric, F.Cu at (170.0, 117.5)
- added C2: 4.7µF, Capacitor_SMD:C_0603_1608Metric, F.Cu at (182.6, 115.7)
- added C4: 4.7µF, Capacitor_SMD:C_0603_1608Metric, F.Cu at (189.5, 114.5)
- added C5: 1uF, Capacitor_SMD:C_0603_1608Metric, F.Cu at (188.0, 113.0)
- added C6: 1uF, Capacitor_SMD:C_0603_1608Metric, F.Cu at (188.8, 116.8)
- added C7: 1u, Capacitor_SMD:C_0603_1608Metric, F.Cu at (173.0, 117.5)
- added C8: 4.7u, Capacitor_SMD:C_0603_1608Metric, F.Cu at (190.5, 85.5)
- added C9: 10pF, Capacitor_SMD:C_0603_1608Metric, F.Cu at (190.5, 109.2)
- added D1: D, Diode_SMD:D_SOD-882D, F.Cu at (171.0, 87.2)
- added D2: D, Diode_SMD:D_SOD-882D, F.Cu at (181.2, 104.0)
- added D3: LED, LED_SMD:LED_0603_1608Metric, F.Cu at (167.0, 86.5)
- added D76: D_Schottky_Small, Diode_SMD:D_0603_1608Metric, F.Cu at (188.0, 87.2)
- added Dig1: KCSA02-105, Display_7Segment:KCSC02-105, F.Cu at (165.5, 95.5)
- added Dig2: KCSA02-105, Display_7Segment:KCSC02-105, F.Cu at (173.0, 95.5)
- added Dig3: KCSA02-105, Display_7Segment:KCSC02-105, F.Cu at (182.0, 95.5)
- added Dig4: KCSA02-105, Display_7Segment:KCSC02-105, F.Cu at (189.5, 95.5)
- added J1: USB_C_Receptacle_USB2.0_14P, Connector_USB:USB_C_Receptacle_HCTL_HC-TYPE-C-16P-01A, F.Cu at (177.5, 83.0)
- added Q1: 2N3904, Package_TO_SOT_SMD:SOT-23, F.Cu at (163.5, 105.8)
- added Q2: 2N3904, Package_TO_SOT_SMD:SOT-23, F.Cu at (167.0, 105.8)
- added Q3: 2N3904, Package_TO_SOT_SMD:SOT-23, F.Cu at (188.0, 105.7)
- added Q4: 2N3904, Package_TO_SOT_SMD:SOT-23, F.Cu at (191.4, 105.7)
- added R1: 27k, Resistor_SMD:R_0201_0603Metric, F.Cu at (170.8, 80.9)
- added R10: 150, Resistor_SMD:R_0603_1608Metric, F.Cu at (171.0, 105.1)
- added R11: 150, Resistor_SMD:R_0603_1608Metric, F.Cu at (184.8, 104.2)
- added R12: 150, Resistor_SMD:R_0603_1608Metric, F.Cu at (191.8, 103.0)
- added R2: 5.1k, Resistor_SMD:R_0603_1608Metric, F.Cu at (184.2, 86.8)
- added R3: 5.1k, Resistor_SMD:R_0603_1608Metric, F.Cu at (170.5, 85.8)
- added R4: 220, Resistor_SMD:R_0603_1608Metric, F.Cu at (163.5, 86.5)
- added R5: 150, Resistor_SMD:R_0603_1608Metric, F.Cu at (163.3, 103.0)
- added R6: 1k, Resistor_SMD:R_0603_1608Metric, F.Cu at (168.0, 109.2)
- added R7: 1k, Resistor_SMD:R_0603_1608Metric, F.Cu at (189.0, 109.2)
- added R8: 1k, Resistor_SMD:R_0603_1608Metric, F.Cu at (164.5, 109.2)
- added R9: 1k, Resistor_SMD:R_0603_1608Metric, F.Cu at (192.5, 109.2)
- added SW1: SW_Push, Button_Switch_SMD:SW_SPST_B3U-1000P, F.Cu at (164.0, 116.0)
- added SW3: SW_Push, Button_Switch_SMD:SW_SPST_B3U-1000P, F.Cu at (164.5, 83.0)
- added SW4: SW_Push, Button_Switch_SMD:SW_SPST_B3U-1000P, F.Cu at (190.5, 83.0)
- added U1: MCP73831-2-OT, Package_TO_SOT_SMD:SOT-23-5, F.Cu at (169.5, 83.0)
- added U3: AP2112K-3.3, Package_TO_SOT_SMD:SOT-23-5, F.Cu at (185.5, 83.0)
- added U7: ATSAMD21E18A-A, Package_QFP:TQFP-32_7x7mm_P0.8mm, F.Cu at (177.5, 110.0)
- added Y2: 32768Hz, Crystal:Crystal_SMD_3215-2Pin_3.2x1.5mm, F.Cu at (169.5, 114.2)
Routing:
- net G: track 0.00 -> 80.8 mm, vias 0 -> 7
- net +5V: track 0.00 -> 80.5 mm
- net F: track 0.00 -> 76.3 mm, vias 0 -> 8
- net A: track 0.00 -> 75.1 mm, vias 0 -> 5
- net B: track 0.00 -> 73.8 mm, vias 0 -> 6
- net D: track 0.00 -> 66.6 mm, vias 0 -> 7
- net E: track 0.00 -> 61.2 mm, vias 0 -> 6
- net C: track 0.00 -> 59.9 mm, vias 0 -> 5
- net DP: track 0.00 -> 56.8 mm, vias 0 -> 5
- net Btn2: track 0.00 -> 46.9 mm, vias 0 -> 2
- net +3.3V: track 0.00 -> 43.9 mm
- net Net-(BT1-+): track 0.00 -> 38.7 mm, vias 0 -> 2
- net Btn1: track 0.00 -> 37.3 mm, vias 0 -> 2
- net A0: track 0.00 -> 30.2 mm, vias 0 -> 2
- net D+: track 0.00 -> 28.9 mm
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- added copper zone on B.Cu, net GND
- added copper zone on F.Cu, net GND
Other:
- board outline added: 34.5 x 38.6 mm
