File: PCB/Watch.kicad_pcb (KiCad board)
At the start: 2 copper layers, 37 x 39.8 mm, 55 parts, among them J1 USB_C_Receptacle_USB2.0_14P, Q1 2N3906, Q2 2N3906, Q3 2N3906, Q4 2N3906, SW1 SW_Push, SW3 SW_Push, SW4 SW_Push, U1 MCP73831-2-OT, U2 TPS63900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

Commit message: Fix regulator and voltage issue, replace inductor with LED
Parts:
- removed C6: 1uF, Capacitor_SMD:C_0402_1005Metric
Connections:
- C5 pad 1: Net-(U7-VDDIN) -> TP_3.3V
- C5 pad 2: TP_3.3V -> GND
- U7 pad 30: Net-(U7-VDDIN) -> TP_3.3V
- U7 pad 9: Net-(U7-VDDANA) -> TP_3.3V
Routing:
- net TP_3.3V: track 71.9 -> 94.8 mm, vias 5 -> 6
- net Net-(U7-VDDANA): track 12.5 -> 0.00 mm, vias 2 -> 0
- net Net-(U7-VDDIN): track 7.26 -> 0.00 mm
